File: Slimmy/Slimmy.kicad_pcb (KiCad board)
At the start: 4 copper layers, 39.2 x 21.2 mm, 22 parts, among them U1 GL3224-OIY04, U2 SD Card, X1 HC-49SMD 25MHZ 20PF 20PPM

Commit message: Final
Other:
- board size 39.2 x 21.2 mm -> 39.2 x 21.5 mm
- board text added: "28 June 2026"
